Commit message: thay đổi code

File: aubo_description/urdf/aubo_i10.xacro (robot description, xacro)
@@ -13,14 +13,14 @@
       <origin xyz="0 0 0" rpy="0 0 0" />
       <geometry>
-        <mesh filename="package://aubo_description/meshes/aubo_i10/visual/link0.DAE" />
-      </geometry>
-      <material name="">
-        <color rgba="1 1 1 1" />
-      </material>
-    </visual>
-    <collision>
-      <origin xyz="0 0 0" rpy="0 0 0" />
-      <geometry>
-        <mesh filename="package://aubo_description/meshes/aubo_i10/collision/link0.STL" />
+        <mesh filename="file://$(find aubo_description)/meshes/aubo_i10/visual/link0.DAE" />
+      </geometry>
+      <material name="">
+        <color rgba="1 1 1 1" />
+      </material>
+    </visual>
+    <collision>
+      <origin xyz="0 0 0" rpy="0 0 0" />
+      <geometry>
+        <mesh filename="file://$(find aubo_description)/meshes/aubo_i10/collision/link0.STL" />
       </geometry>
     </collision>
@@ -36,5 +36,5 @@
       <geometry>
         <mesh
-          filename="package://aubo_description/meshes/aubo_i10/visual/link1.DAE" />
+          filename="file://$(find aubo_description)/meshes/aubo_i10/visual/link1.DAE" />
       </geometry>
       <material name="">
@@ -45,5 +45,5 @@
       <origin xyz="0 0 0" rpy="0 0 0" />
       <geometry>
-        <mesh filename="package://aubo_description/meshes/aubo_i10/collision/link1.STL" />
+        <mesh filename="file://$(find aubo_description)/meshes/aubo_i10/collision/link1.STL" />
       </geometry>
     </collision>
@@ -66,5 +66,5 @@
       <origin xyz="0 0 0" rpy="0 0 0" />
       <geometry>
-        <mesh filename="package://aubo_description/meshes/aubo_i10/visual/link2.DAE" />
+        <mesh filename="file://$(find aubo_description)/meshes/aubo_i10/visual/link2.DAE" />
       </geometry>
       <material name="">
@@ -75,5 +75,5 @@
       <origin xyz="0 0 0" rpy="0 0 0" />
       <geometry>
-        <mesh filename="package://aubo_description/meshes/aubo_i10/collision/link2.STL" />
+        <mesh filename="file://$(find aubo_description)/meshes/aubo_i10/collision/link2.STL" />
       </geometry>
     </collision>
@@ -96,14 +96,14 @@
       <origin xyz="0 0 0" rpy="0 0 0" />
       <geometry>
-        <mesh filename="package://aubo_description/meshes/aubo_i10/visual/link3.DAE" />
-      </geometry>
-      <material name="">
-        <color rgba="1 1 1 1" />
-      </material>
-    </visual>
-    <collision>
-      <origin xyz="0 0 0" rpy="0 0 0" />
-      <geometry>
-        <mesh filename="package://aubo_description/meshes/aubo_i10/collision/link3.STL" />
+        <mesh filename="file://$(find aubo_description)/meshes/aubo_i10/visual/link3.DAE" />
+      </geometry>
+      <material name="">
+        <color rgba="1 1 1 1" />
+      </material>
+    </visual>
+    <collision>
+      <origin xyz="0 0 0" rpy="0 0 0" />
+      <geometry>
+        <mesh filename="file://$(find aubo_description)/meshes/aubo_i10/collision/link3.STL" />
       </geometry>
     </collision>
@@ -126,14 +126,14 @@
       <origin xyz="0 0 0" rpy="0 0 0" />
       <geometry>
-        <mesh filename="package://aubo_description/meshes/aubo_i10/visual/link4.DAE" />
-      </geometry>
-      <material name="">
-        <color rgba="1 1 1 1" />
-      </material>
-    </visual>
-    <collision>
-      <origin xyz="0 0 0" rpy="0 0 0" />
-      <geometry>
-        <mesh filename="package://aubo_description/meshes/aubo_i10/collision/link4.STL" />
+        <mesh filename="file://$(find aubo_description)/meshes/aubo_i10/visual/link4.DAE" />
+      </geometry>
+      <material name="">
+        <color rgba="1 1 1 1" />
+      </material>
+    </visual>
+    <collision>
+      <origin xyz="0 0 0" rpy="0 0 0" />
+      <geometry>
+        <mesh filename="file://$(find aubo_description)/meshes/aubo_i10/collision/link4.STL" />
       </geometry>
     </collision>
@@ -156,14 +156,14 @@
       <origin xyz="0 0 0" rpy="0 0 0" />
       <geometry>
-        <mesh filename="package://aubo_description/meshes/aubo_i10/visual/link5.DAE" />
-      </geometry>
-      <material name="">
-        <color rgba="1 1 1 1" />
-      </material>
-    </visual>
-    <collision>
-      <origin xyz="0 0 0" rpy="0 0 0" />
-      <geometry>
-        <mesh filename="package://aubo_description/meshes/aubo_i10/collision/link5.STL" />
+        <mesh filename="file://$(find aubo_description)/meshes/aubo_i10/visual/link5.DAE" />
+      </geometry>
+      <material name="">
+        <color rgba="1 1 1 1" />
+      </material>
+    </visual>
+    <collision>
+      <origin xyz="0 0 0" rpy="0 0 0" />
+      <geometry>
+        <mesh filename="file://$(find aubo_description)/meshes/aubo_i10/collision/link5.STL" />
       </geometry>
     </collision>
@@ -186,14 +186,14 @@
       <origin xyz="0 0 0" rpy="0 0 0" />
       <geometry>
-        <mesh filename="package://aubo_description/meshes/aubo_i10/visual/link6.DAE" />
-      </geometry>
-      <material name="">
-        <color rgba="1 1 1 1" />
-      </material>
-    </visual>
-    <collision>
-      <origin xyz="0 0 0" rpy="0 0 0" />
-      <geometry>
-        <mesh filename="package://aubo_description/meshes/aubo_i10/collision/link6.STL" />
+        <mesh filename="file://$(find aubo_description)/meshes/aubo_i10/visual/link6.DAE" />
+      </geometry>
+      <material name="">
+        <color rgba="1 1 1 1" />
+      </material>
+    </visual>
+    <collision>
+      <origin xyz="0 0 0" rpy="0 0 0" />
+      <geometry>
+        <mesh filename="file://$(find aubo_description)/meshes/aubo_i10/collision/link6.STL" />
       </geometry>
     </collision>

File: aubo_description/urdf/aubo_i10_dh_ag95.xacro (robot description, xacro)
@@ -6,5 +6,5 @@
 <xacro:property name="fingerprefix" value="$(arg fingerprefix)"/>
   <!-- Include file robot gốc và file macro gripper -->
-  <xacro:include filename="$(find aubo_description)/urdf/aubo_i10.urdf" />
+  <xacro:include filename="$(find aubo_description)/urdf/aubo_i10.xacro" />
   <xacro:include filename="$(find aubo_description)/urdf/dh_ag95_macro.xacro" />
   <xacro:include filename="$(find aubo_description)/urdf/ros2_control.xacro" />

File: aubo_description/urdf/dh_ag95_macro.xacro (robot description, xacro)
@@ -29,5 +29,5 @@
           <origin xyz="-0.036673 0.00875 -0.098336" rpy="0 0 0" />
           <geometry>
-            <mesh filename="package://aubo_description/meshes/aubo_i10/visual/outer_knuckle.stl"
+            <mesh filename="file://$(find aubo_description)/meshes/aubo_i10/visual/outer_knuckle.stl"
               scale="0.001 0.001 0.001" />
           </geometry>
@@ -39,5 +39,5 @@
           <origin xyz="-0.036673 0.00875 -0.098336" rpy="0 0 0" />
           <geometry>
-            <mesh filename="package://aubo_description/meshes/aubo_i10/collision/outer_knuckle.stl"
+            <mesh filename="file://$(find aubo_description)/meshes/aubo_i10/collision/outer_knuckle.stl"
               scale="0.001 0.001 0.001" />
           </geometry>
@@ -60,5 +60,5 @@
           <origin xyz="-0.016 0.0254 -0.10586" rpy="0 0 0" />
           <geometry>
-            <mesh filename="package://aubo_description/meshes/aubo_i10/visual/inner_knuckle.stl"
+            <mesh filename="file://$(find aubo_description)/meshes/aubo_i10/visual/inner_knuckle.stl"
               scale="0.001 0.001 0.001" />
           </geometry>
@@ -70,5 +70,5 @@
           <origin xyz="-0.016 0.0254 -0.10586" rpy="0 0 0" />
           <geometry>
-            <mesh filename="package://aubo_description/meshes/aubo_i10/collision/inner_knuckle.stl"
+            <mesh filename="file://$(find aubo_description)/meshes/aubo_i10/collision/inner_knuckle.stl"
               scale="0.001 0.001 0.001" />
           </geometry>
@@ -91,5 +91,5 @@
           <origin xyz="-0.091673 0.00875 -0.098336" rpy="0 0 0" />
           <geometry>
-            <mesh filename="package://aubo_description/meshes/aubo_i10/visual/finger.stl"
+            <mesh filename="file://$(find aubo_description)/meshes/aubo_i10/visual/finger.stl"
               scale="0.001 0.001 0.001" />
           </geometry>
@@ -101,5 +101,5 @@
           <origin xyz="-0.091673 0.00875 -0.098336" rpy="0 0 0" />
           <geometry>
-            <mesh filename="package://aubo_description/meshes/aubo_i10/collision/finger.stl"
+            <mesh filename="file://$(find aubo_description)/meshes/aubo_i10/collision/finger.stl"
               scale="0.001 0.001 0.001" />
           </geometry>
@@ -124,5 +124,5 @@
           <origin xyz="-0.0705 -0.0 -0.12056" rpy="0 0 0" />
           <geometry>
-            <mesh filename="package://aubo_description/meshes/aubo_i10/visual/finger_pad.stl"
+            <mesh filename="file://$(find aubo_description)/meshes/aubo_i10/visual/finger_pad.stl"
               scale="0.001 0.001 0.001" />
           </geometry>
@@ -134,5 +134,5 @@
           <origin xyz="-0.0705 -0.0 -0.12056" rpy="0 0 0" />
           <geometry>
-            <mesh filename="package://aubo_description/meshes/aubo_i10/collision/finger_pad.stl"
+            <mesh filename="file://$(find aubo_description)/meshes/aubo_i10/collision/finger_pad.stl"
               scale="0.001 0.001 0.001" />
           </geometry>
@@ -215,5 +215,5 @@
         <origin xyz="0 0 0" rpy="0 0 0" />
         <geometry>
-          <mesh filename="package://aubo_description/meshes/aubo_i10/visual/base_link.stl"
+          <mesh filename="file://$(find aubo_description)/meshes/aubo_i10/visual/base_link.stl"
             scale="0.001 0.001 0.001" />
         </geometry>
@@ -225,5 +225,5 @@
         <origin xyz="0 0 0" rpy="0 0 0" />
         <geometry>
-          <mesh filename="package://aubo_description/meshes/aubo_i10/collision/base_link.stl"
+          <mesh filename="file://$(find aubo_description)/meshes/aubo_i10/collision/base_link.stl"
             scale="0.001 0.001 0.001" />
         </geometry>
@@ -245,5 +245,5 @@
         <origin xyz="0.0405 0.0143 -0.0147" rpy="0 0 0" />
         <geometry>
-          <mesh filename="package://aubo_description/meshes/aubo_i10/visual/gripper_body.stl"
+          <mesh filename="file://$(find aubo_description)/meshes/aubo_i10/visual/gripper_body.stl"
             scale="0.001 0.001 0.001" />
         </geometry>
@@ -255,5 +255,5 @@
         <origin xyz="0.0405 0.0143 -0.0147" rpy="0 0 0" />
         <geometry>
-          <mesh filename="package://aubo_description/meshes/aubo_i10/collision/gripper_body.stl"
+          <mesh filename="file://$(find aubo_description)/meshes/aubo_i10/collision/gripper_body.stl"
             scale="0.001 0.001 0.001" />
         </geometry>
